Commit message: [Aerial Handover] add collision model for hand

File: aerial_handover/urdf/hand.urdf.xacro (robot description, xacro)
@@ -10,7 +10,13 @@
       <origin xyz="0 0 0" rpy="-1.5708 0 -1.5708"/>
       <geometry>
-          <mesh filename="package://aerial_handover/urdf/mesh/hand.dae" scale= "0.01 0.01 0.01"/>
+        <mesh filename="package://aerial_handover/urdf/mesh/hand.dae" scale= "0.01 0.01 0.01"/>
       </geometry>
     </visual>
+    <collision>
+      <origin xyz="0 0 0" rpy="-1.5708 0 -1.5708"/>
+      <geometry>
+          <box size="0.1 0.05 0.2" />
+      </geometry>
+    </collision>
   </link>
   <gazebo reference="hand_link">
